File: E_Veveris_MultiVib/E_Veveris_MultiVib.sch (KiCad schematic (older format))
At the start: 11 parts

Commit message: 3 lekcijas uzdevums
Parts:
- removed Q? (x2): BC548, Package_TO_SOT_THT:TO-92_Inline, symbol Transistor_BJT:BC548
- added U1: BC846BDW1T1G, symbol MultiVib_Libary:BC846BDW1T1G
- gave numbers to parts that had none: 9
Connections:
- net at BT1.2 (-): now also U1.1 (E_TR2), U1.4 (E_TR1)
- net at C1.1, R1.2: now also U1.3 (C_TR1)
- net at C1.2, R2.2: now also U1.2 (B_TR2)
- net at C2.2, R3.2: now also U1.5 (B_TR1)
- net at C2.1, R4.2: now also U1.6 (C_TR2)
Other:
- moved on the sheet: C2, D2, R3, R4
Changed lines of the file:
@@
 EESchema Schematic File Version 4
+LIBS:E_Veveris_MultiVib-cache
 EELAYER 30 0
 EELAYER END
@@
 $EndDescr
 $Comp
-L Device:Battery BT?
+L Device:Battery BT1
 U 1 1 5E56FC33
 P 3100 3400
-F 0 "BT?" H 3208 3446 50  0000 L CNN
+F 0 "BT1" H 3208 3446 50  0000 L CNN
 F 1 "9V" H 3208 3355 50  0000 L CNN
 F 2 "" V 3100 3460 50  0001 C CNN
@@
 $EndComp
 $Comp
-L Device:R R?
+L Device:R R1
 U 1 1 5E570027
 P 3550 3100
-F 0 "R?" H 3620 3146 50  0000 L CNN
+F 0 "R1" H 3620 3146 50  0000 L CNN
 F 1 "470R" V 3550 3000 50  0000 L CNN
 F 2 "" V 3480 3100 50  0001 C CNN
@@
 $EndComp
 $Comp
-L Device:R R?
+L Device:R R2
 U 1 1 5E5705D7
 P 3950 3100
-F 0 "R?" H 4020 3146 50  0000 L CNN
+F 0 "R2" H 4020 3146 50  0000 L CNN
 F 1 "47K" V 3950 3050 50  0000 L CNN
 F 2 "" V 3880 3100 50  0001 C CNN
@@
 $EndComp
 $Comp
-L Device:R R?
+L Device:R R3
 U 1 1 5E5706BD
-P 4400 3100
-F 0 "R?" H 4470 3146 50  0000 L CNN
-F 1 "47K" V 4400 3050 50  0000 L CNN
-F 2 "" V 4330 3100 50  0001 C CNN
-F 3 "~" H 4400 3100 50  0001 C CNN
-	1    4400 3100
-	1    0    0    -1
-$EndComp
-$Comp
-L Device:R R?
+P 5200 3100
+F 0 "R3" H 5270 3146 50  0000 L CNN
+F 1 "47K" V 5200 3050 50  0000 L CNN
+F 2 "" V 5130 3100 50  0001 C CNN
+F 3 "~" H 5200 3100 50  0001 C CNN
+	1    5200 3100
+	1    0    0    -1
+$EndComp
+$Comp
+L Device:R R4
 U 1 1 5E57091C
-P 4800 3100
-F 0 "R?" H 4870 3146 50  0000 L CNN
-F 1 "470R" V 4800 3000 50  0000 L CNN
-F 2 "" V 4730 3100 50  0001 C CNN
-F 3 "~" H 4800 3100 50  0001 C CNN
-	1    4800 3100
-	1    0    0    -1
-$EndComp
-$Comp
-L Device:LED D?
+P 5600 3100
+F 0 "R4" H 5670 3146 50  0000 L CNN
+F 1 "470R" V 5600 3000 50  0000 L CNN
+F 2 "" V 5530 3100 50  0001 C CNN
+F 3 "~" H 5600 3100 50  0001 C CNN
+	1    5600 3100
+	1    0    0    -1
+$EndComp
+$Comp
+L Device:LED D1
 U 1 1 5E570C13
 P 3550 2550
-F 0 "D?" V 3589 2433 50  0000 R CNN
+F 0 "D1" V 3589 2433 50  0000 R CNN
 F 1 "LED" V 3498 2433 50  0000 R CNN
 F 2 "" H 3550 2550 50  0001 C CNN
@@
 $EndComp
 $Comp
-L Device:LED D?
+L Device:LED D2
 U 1 1 5E57169A
-P 4800 2550
-F 0 "D?" V 4839 2433 50  0000 R CNN
-F 1 "LED" V 4748 2433 50  0000 R CNN
-F 2 "" H 4800 2550 50  0001 C CNN
-F 3 "~" H 4800 2550 50  0001 C CNN
-	1    4800 2550
+P 5600 2550
+F 0 "D2" V 5639 2433 50  0000 R CNN
+F 1 "LED" V 5548 2433 50  0000 R CNN
+F 2 "" H 5600 2550 50  0001 C CNN
+F 3 "~" H 5600 2550 50  0001 C CNN
+	1    5600 2550
 	0    -1   -1   0
 $EndComp
 Wire Wire Line
-	4800 2700 4800 2950
+	5600 2700 5600 2950
 Wire Wire Line
 	3550 2950 3550 2700
@@
 	3550 2200 3550 2400
 Wire Wire Line
-	4400 2950 4400 2200
-Wire Wire Line
-	4400 2200 3950 2200
-Connection ~ 3950 2200
-Wire Wire Line
-	4800 2400 4800 2200
-Wire Wire Line
-	4800 2200 4400 2200
-Connection ~ 4400 2200
-$Comp
-L Device:CP1 C?
+	5200 2950 5200 2200
+Wire Wire Line
+	5600 2400 5600 2200
+$Comp
+L Device:CP1 C1
 U 1 1 5E572C93
 P 3750 3450
-F 0 "C?" V 4002 3450 50  0000 C CNN
+F 0 "C1" V 4002 3450 50  0000 C CNN
 F 1 "47uF" V 3911 3450 50  0000 C CNN
 F 2 "" H 3750 3450 50  0001 C CNN
@@
 $EndComp
 $Comp
-L Device:CP1 C?
+L Device:CP1 C2
 U 1 1 5E5732B6
-P 4600 3450
-F 0 "C?" V 4348 3450 50  0000 C CNN
-F 1 "47uF" V 4439 3450 50  0000 C CNN
-F 2 "" H 4600 3450 50  0001 C CNN
-F 3 "~" H 4600 3450 50  0001 C CNN
-	1    4600 3450
+P 5400 3450
+F 0 "C2" V 5148 3450 50  0000 C CNN
+F 1 "47uF" V 5239 3450 50  0000 C CNN
+F 2 "" H 5400 3450 50  0001 C CNN
+F 3 "~" H 5400 3450 50  0001 C CNN
+	1    5400 3450
 	0    1    1    0
 $EndComp
 Wire Wire Line
-	4800 3250 4800 3450
-Wire Wire Line
-	4800 3450 4750 3450
-Wire Wire Line
-	4400 3250 4400 3450
-Wire Wire Line
-	4400 3450 4450 3450
+	5600 3250 5600 3450
+Wire Wire Line
+	5600 3450 5550 3450
+Wire Wire Line
+	5200 3250 5200 3450
+Wire Wire Line
+	5200 3450 5250 3450
 Wire Wire Line
 	3900 3450 3950 3450
@@
 Wire Wire Line
 	3550 3450 3550 3250
-$Comp
-L Transistor_BJT:BC548 Q?
-U 1 1 5E5742D0
-P 4700 3900
-F 0 "Q?" H 4891 3946 50  0000 L CNN
-F 1 "BC548" H 4891 3855 50  0000 L CNN
-F 2 "Package_TO_SOT_THT:TO-92_Inline" H 4900 3825 50  0001 L CIN
-F 3 "http://www.fairchildsemi.com/ds/BC/BC547.pdf" H 4700 3900 50  0001 L CNN
-	1    4700 3900
-	1    0    0    -1
-$EndComp
-$Comp
-L Transistor_BJT:BC548 Q?
-U 1 1 5E574CC4
-P 3650 3850
-F 0 "Q?" H 3841 3896 50  0000 L CNN
-F 1 "BC548" H 3841 3805 50  0000 L CNN
-F 2 "Package_TO_SOT_THT:TO-92_Inline" H 3850 3775 50  0001 L CIN
-F 3 "http://www.fairchildsemi.com/ds/BC/BC547.pdf" H 3650 3850 50  0001 L CNN
-	1    3650 3850
-	-1   0    0    -1
-$EndComp
-Wire Wire Line
-	3550 3650 3550 3450
-Connection ~ 3550 3450
-Wire Wire Line
-	4800 3700 4800 3450
-Connection ~ 4800 3450
-Wire Wire Line
-	3850 3850 4400 3850
-Wire Wire Line
-	4400 3850 4400 3450
-Connection ~ 4400 3450
-Wire Wire Line
-	4500 3900 3950 3900
-Wire Wire Line
-	3950 3900 3950 3450
-Connection ~ 3950 3450
+Connection ~ 5600 3450
 Wire Wire Line
 	3100 3200 3100 2200
@@
 Wire Wire Line
 	3100 3600 3100 4200
-Wire Wire Line
-	3100 4200 3550 4200
-Wire Wire Line
-	3550 4200 3550 4050
-Wire Wire Line
-	3550 4200 4800 4200
-Wire Wire Line
-	4800 4200 4800 4100
-Connection ~ 3550 4200
+$Comp
+L MultiVib_Libary:BC846BDW1T1G U1
+U 1 1 5E5F998A
+P 4450 3800
+F 0 "U1" H 4450 4000 50  0000 C CNN
+F 1 "BC846BDW1T1G" H 4450 3450 50  0000 C CNN
+F 2 "" H 4450 4000 50  0001 C CNN
+F 3 "" H 4450 4000 50  0001 C CNN
+	1    4450 3800
+	1    0    0    -1
+$EndComp
+Wire Wire Line
+	3550 4050 3550 3450
+Connection ~ 3550 3450
+Connection ~ 5200 3450
+Wire Wire Line
+	5600 3450 5600 3750
+Connection ~ 3950 3450
+Connection ~ 5200 2200
+Wire Wire Line
+	5200 3450 5200 3900
+Wire Wire Line
+	5200 2200 5600 2200
+Wire Wire Line
+	4850 3900 5200 3900
+Wire Wire Line
+	4850 3750 5600 3750
+Wire Wire Line
+	4050 3900 3950 3900
+Wire Wire Line
+	3950 3450 3950 3900
+Wire Wire Line
+	3550 4050 4050 4050
+Wire Wire Line
+	4050 3750 4000 3750
+Wire Wire Line
+	4000 3750 4000 4200
+Connection ~ 4000 4200
+Wire Wire Line
+	4850 4200 4850 4050
+Wire Wire Line
+	4000 4200 4850 4200
+Wire Wire Line
+	3100 4200 4000 4200
+Wire Wire Line
+	3950 2200 5200 2200
+Connection ~ 3950 2200
 $EndSCHEMATC
