File: PWR_Supply/PWR_Supply/PWR_Supply.sch (KiCad schematic (older format))
At the start: 5 parts, among them J1 220VAC, J2 12V_OUT, J3 5V_OUT, J4 9V_OUT, J5 3,3V_OUT

Commit message: Pabeigts majasdarbs
Parts:
- removed J2: 12V_OUT, symbol Connector:Screw_Terminal_01x02
- removed J3: 5V_OUT, symbol Connector:Screw_Terminal_01x02
- removed J4: 9V_OUT, symbol Connector:Screw_Terminal_01x02
- removed J5: 3,3V_OUT, symbol Connector:Screw_Terminal_01x02
- added J?: Conn_01x05, symbol Connector_Generic:Conn_01x05
Connections:
- net GNDREF: now also J?.5 (Pin_5)
- new net 12V: J?.4 (Pin_4)
- new net 3,3V: J?.1 (Pin_1)
- new net 5V: J?.2 (Pin_2)
- new net 9V: J?.3 (Pin_3)
Changed lines of the file:
@@
 EESchema Schematic File Version 4
+LIBS:PWR_Supply-cache
 EELAYER 30 0
 EELAYER END
@@
 	4150 2350 3800 2350
 Wire Wire Line
-	3800 2350 3800 1550
-Wire Wire Line
-	3800 1550 3750 1550
+	3800 2350 3800 2150
 Wire Wire Line
 	4150 1550 3800 1550
 Connection ~ 3800 1550
-Wire Wire Line
-	4700 1550 4850 1550
 $Comp
 L power:GNDREF #PWR03
@@
 Wire Wire Line
 	5050 1800 5150 1800
-$Comp
-L Connector:Screw_Terminal_01x02 J5
-U 1 1 5E712F70
-P 6250 1550
-F 0 "J5" H 6330 1542 50  0000 L CNN
-F 1 "3,3V_OUT" H 6330 1451 50  0000 L CNN
-F 2 "" H 6250 1550 50  0001 C CNN
-F 3 "~" H 6250 1550 50  0001 C CNN
-	1    6250 1550
-	1    0    0    -1
-$EndComp
-$Comp
-L Connector:Screw_Terminal_01x02 J3
-U 1 1 5E71357E
-P 4850 1050
-F 0 "J3" V 4814 862 50  0000 R CNN
-F 1 "5V_OUT" V 4723 862 50  0000 R CNN
-F 2 "" H 4850 1050 50  0001 C CNN
-F 3 "~" H 4850 1050 50  0001 C CNN
-	1    4850 1050
-	0    -1   -1   0
-$EndComp
-$Comp
-L Connector:Screw_Terminal_01x02 J4
-U 1 1 5E713BB9
-P 5350 2350
-F 0 "J4" H 5430 2342 50  0000 L CNN
-F 1 "9V_OUT" H 5430 2251 50  0000 L CNN
-F 2 "" H 5350 2350 50  0001 C CNN
-F 3 "~" H 5350 2350 50  0001 C CNN
-	1    5350 2350
-	1    0    0    -1
-$EndComp
-$Comp
-L Connector:Screw_Terminal_01x02 J2
-U 1 1 5E713F3A
-P 3750 1050
-F 0 "J2" V 3714 862 50  0000 R CNN
-F 1 "12V_OUT" V 3623 862 50  0000 R CNN
-F 2 "" H 3750 1050 50  0001 C CNN
-F 3 "~" H 3750 1050 50  0001 C CNN
-	1    3750 1050
-	0    -1   -1   0
-$EndComp
 $Comp
 L Connector:Screw_Terminal_01x02 J1
@@
 Wire Wire Line
 	1300 1600 1500 1600
-Wire Wire Line
-	3750 1250 3750 1550
-Connection ~ 3750 1550
-Wire Wire Line
-	3750 1550 3550 1550
-Wire Wire Line
-	4850 1250 4850 1550
-Connection ~ 4850 1550
-Wire Wire Line
-	4850 1550 5150 1550
-Wire Wire Line
-	5150 2350 4700 2350
-Wire Wire Line
-	6050 1550 5700 1550
-$Comp
-L power:GNDREF #PWR07
-U 1 1 5E7159F6
-P 6050 1750
-F 0 "#PWR07" H 6050 1500 50  0001 C CNN
-F 1 "GNDREF" H 6055 1577 50  0000 C CNN
-F 2 "" H 6050 1750 50  0001 C CNN
-F 3 "" H 6050 1750 50  0001 C CNN
-	1    6050 1750
-	1    0    0    -1
-$EndComp
-$Comp
-L power:GNDREF #PWR04
-U 1 1 5E715ED3
-P 4950 1350
-F 0 "#PWR04" H 4950 1100 50  0001 C CNN
-F 1 "GNDREF" H 4955 1177 50  0000 C CNN
-F 2 "" H 4950 1350 50  0001 C CNN
-F 3 "" H 4950 1350 50  0001 C CNN
-	1    4950 1350
-	1    0    0    -1
-$EndComp
-$Comp
-L power:GNDREF #PWR02
-U 1 1 5E71600E
-P 3850 1350
-F 0 "#PWR02" H 3850 1100 50  0001 C CNN
-F 1 "GNDREF" H 3855 1177 50  0000 C CNN
-F 2 "" H 3850 1350 50  0001 C CNN
-F 3 "" H 3850 1350 50  0001 C CNN
-	1    3850 1350
-	1    0    0    -1
-$EndComp
-$Comp
-L power:GNDREF #PWR06
-U 1 1 5E71630A
-P 5150 2550
-F 0 "#PWR06" H 5150 2300 50  0001 C CNN
-F 1 "GNDREF" H 5155 2377 50  0000 C CNN
-F 2 "" H 5150 2550 50  0001 C CNN
-F 3 "" H 5150 2550 50  0001 C CNN
-	1    5150 2550
-	1    0    0    -1
-$EndComp
-Wire Wire Line
-	6050 1750 6050 1650
-Wire Wire Line
-	5150 2550 5150 2450
-Wire Wire Line
-	4950 1350 4950 1250
-Wire Wire Line
-	3850 1350 3850 1250
+Entry Wire Line
+	6200 2050 6100 1950
+Entry Wire Line
+	6200 2000 6100 1900
+Entry Wire Line
+	6200 1950 6100 1850
+Text Label 7850 1300 0    50   ~ 0
+3,3V
+Text Label 7850 1400 0    50   ~ 0
+5V
+Text Label 7850 1500 0    50   ~ 0
+9V
+Text Label 7850 1600 0    50   ~ 0
+12V
+Text Label 3600 1550 0    50   ~ 0
+12V
+Text Label 4750 1550 0    50   ~ 0
+5V
+Entry Wire Line
+	6200 1900 6100 1800
+$Comp
+L Connector_Generic:Conn_01x05 J?
+U 1 1 5E71D81F
+P 8200 1500
+F 0 "J?" H 8280 1542 50  0000 L CNN
+F 1 "Conn_01x05" H 8280 1451 50  0000 L CNN
+F 2 "" H 8200 1500 50  0001 C CNN
+F 3 "~" H 8200 1500 50  0001 C CNN
+	1    8200 1500
+	1    0    0    -1
+$EndComp
+Text GLabel 6200 2050 2    50   Input ~ 0
+Power_BUS
+Entry Wire Line
+	7650 1500 7750 1600
+Entry Wire Line
+	7650 1400 7750 1500
+Entry Wire Line
+	7650 1300 7750 1400
+Entry Wire Line
+	7650 1200 7750 1300
+Text GLabel 7650 1200 0    50   Input ~ 0
+Power_BUS
+Wire Wire Line
+	8000 1300 7750 1300
+Wire Wire Line
+	7750 1400 8000 1400
+Wire Wire Line
+	8000 1500 7750 1500
+Wire Wire Line
+	7750 1600 8000 1600
+$Comp
+L power:GNDREF #PWR?
+U 1 1 5E72B168
+P 8000 1800
+F 0 "#PWR?" H 8000 1550 50  0001 C CNN
+F 1 "GNDREF" H 8005 1627 50  0000 C CNN
+F 2 "" H 8000 1800 50  0001 C CNN
+F 3 "" H 8000 1800 50  0001 C CNN
+	1    8000 1800
+	1    0    0    -1
+$EndComp
+Wire Wire Line
+	8000 1700 8000 1800
+Wire Wire Line
+	3550 1550 3800 1550
+Wire Wire Line
+	4700 1550 4950 1550
+Wire Wire Line
+	5700 1550 5850 1550
+Wire Wire Line
+	5850 1550 5850 1950
+Wire Wire Line
+	5850 1950 6100 1950
+Wire Wire Line
+	6100 1900 5900 1900
+Wire Wire Line
+	5900 1350 4950 1350
+Wire Wire Line
+	4950 1350 4950 1550
+Wire Wire Line
+	5900 1350 5900 1900
+Connection ~ 4950 1550
+Wire Wire Line
+	4950 1550 5150 1550
+Wire Wire Line
+	6100 1850 5800 1850
+Wire Wire Line
+	5800 1850 5800 2350
+Wire Wire Line
+	5800 2350 4700 2350
+Wire Wire Line
+	6100 1800 5750 1800
+Wire Wire Line
+	5750 1800 5750 2150
+Wire Wire Line
+	5750 2150 3800 2150
+Wire Bus Line
+	7650 1200 7650 1550
+Wire Bus Line
+	6200 1750 6200 2050
+Connection ~ 3800 2150
+Wire Wire Line
+	3800 2150 3800 1550
 $EndSCHEMATC
