File: Battery/_autosave-Battery.sch (KiCad schematic (older format))
At the start: 1 part

Commit message: Mājas darbs
Parts:
- added R1: R, Resistor_SMD:R_0805_2012Metric, symbol Device:R
- BT1: renamed from BT?; footprint (none) -> Battery_Holder:S8211R
Connections:
- net at BT1.1 (+): now also R1.1
- net at BT1.2 (-): now also R1.2
Changed lines of the file:
@@
 $EndDescr
 $Comp
-L Device:Battery_Cell BT?
+L Device:Battery_Cell BT1
 U 1 1 5E7B0D08
 P 5550 3700
-F 0 "BT?" H 5668 3796 50  0000 L CNN
+F 0 "BT1" H 5668 3796 50  0000 L CNN
 F 1 "Battery_Cell" H 5668 3705 50  0000 L CNN
-F 2 "" V 5550 3760 50  0001 C CNN
+F 2 "Battery_Holder:S8211R" V 5550 3760 50  0001 C CNN
 F 3 "~" V 5550 3760 50  0001 C CNN
 	1    5550 3700
 	1    0    0    -1
 $EndComp
+$Comp
+L Device:R R1
+U 1 1 5E7B1102
+P 5200 3650
+F 0 "R1" H 5270 3696 50  0000 L CNN
+F 1 "R" H 5270 3605 50  0000 L CNN
+F 2 "Resistor_SMD:R_0805_2012Metric" V 5130 3650 50  0001 C CNN
+F 3 "~" H 5200 3650 50  0001 C CNN
+	1    5200 3650
+	1    0    0    -1
+$EndComp
+Wire Wire Line
+	5550 3500 5550 3400
+Wire Wire Line
+	5550 3400 5200 3400
+Wire Wire Line
+	5200 3400 5200 3500
+Wire Wire Line
+	5200 3800 5200 3950
+Wire Wire Line
+	5200 3950 5550 3950
+Wire Wire Line
+	5550 3950 5550 3800
 $EndSCHEMATC
