File: Single_Transistor_AMP/Single_Transitor_Amp/Single_Transitor_Amp.kicad_pcb (KiCad board)
At the start: 4 copper layers, 0 parts

Commit message: 15.04 Lekcijas Mājas darbs
Parts:
- added BT1: 3V, Connector_PinHeader_1.27mm:PinHeader_1x02_P1.27mm_Vertical, F.Cu at (113.2, 104.5)
- added C1: 1uF, Capacitor_THT:CP_Radial_D6.3mm_P2.50mm, F.Cu at (106.4, 114.0)
- added C2: 4,7nF, Capacitor_SMD:C_0603_1608Metric, F.Cu at (116.4, 109.7)
- added C3: 10nF, Capacitor_SMD:C_1206_3216Metric, F.Cu at (107.7, 107.4)
- added J1: Signal_IN, Connector_PinHeader_1.27mm:PinHeader_1x02_P1.27mm_Vertical, F.Cu at (103.2, 109.3)
- added J2: Signal_Out, Connector_PinHeader_1.27mm:PinHeader_1x02_P1.27mm_Vertical, F.Cu at (120.9, 110.1)
- added Q1: BC547, Package_TO_SOT_THT:TO-92, F.Cu at (114.1, 108.3)
- added R1: 820K, Resistor_SMD:R_0603_1608Metric, F.Cu at (118.0, 109.7)
- added R2: 22, Resistor_SMD:R_0603_1608Metric, F.Cu at (108.4, 109.3)
Other:
- board outline added: 24.2 x 15.9 mm
- net class Power: trace_width 0.7 -> 0.4

Commit message: 22.04 Lekcijas M.D
Parts:
- moved R2 1.39 mm to (107.0, 109.4)
Routing:
- net Net-(C2-Pad1): track 0.00 -> 14.1 mm
- net Net-(BT1-Pad2): track 0.00 -> 12.7 mm
- net Net-(C1-Pad2): track 0.00 -> 12.2 mm
- net Net-(BT1-Pad1): track 0.00 -> 9.45 mm
- net Net-(C1-Pad1): track 0.00 -> 4.73 mm
- net Net-(Q1-Pad3): track 0.00 -> 4.16 mm
- added copper zone on F.Cu, net (none)
- added copper zone on B.Cu, net Net-(BT1-Pad1)
- added copper zone on F.Cu, net Net-(BT1-Pad1)
Changed lines of the file:
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@@
     (thickness 1.6)
     (drawings 4)
-    (tracks 0)
+    (tracks 30)
     (zones 0)
     (modules 9)
@@
   (setup
     (last_trace_width 0.25)
+    (user_trace_width 0.4)
+    (user_trace_width 0.5)
+    (user_trace_width 0.6)
     (trace_clearance 0.2)
     (zone_clearance 0.508)
@@
   )
   (module Resistor_SMD:R_0603_1608Metric placed (layer F.Cu)
-    (at 108.44 109.34 180)
+    (at 107.05 109.37 180)
     (descr "Resistor SMD 0603 (1608 Metric), square (rectangular) end terminal, IPC_7351 nominal, (Body size source: http://www.tortai-tech.com/upload/download/2011102023233369053.pdf), generated with kicad-footprint-generator")
     (tags resistor)
     (attr smd)
-    (fp_text reference R2 (at 2.63 -0.18) (layer F.SilkS)
+    (fp_text reference R2 (at -2.5 -0.05) (layer F.SilkS)
       (effects (font (size 1 1) (thickness 0.15)))
     )
@@
   (gr_line (start 102.685733 117.834348) (end 119.61 117.84) (layer Edge.Cuts) (width 0.05))
   (gr_line (start 120.810837 101.949371) (end 101.49 101.95) (layer Edge.Cuts) (width 0.05))
+  (segment (start 116.52 104.5) (end 113.24 104.5) (width 0.5) (layer F.Cu) (net 1))
+  (segment (start 120.88 108.86) (end 116.52 104.5) (width 0.5) (layer F.Cu) (net 1))
+  (segment (start 109.14 104.5) (end 106.25 107.39) (width 0.5) (layer F.Cu) (net 2))
+  (segment (start 111.97 104.5) (end 109.14 104.5) (width 0.5) (layer F.Cu) (net 2))
+  (segment (start 105.11 107.39) (end 103.22 109.28) (width 0.5) (layer F.Cu) (net 2))
+  (segment (start 106.25 107.39) (end 105.11 107.39) (width 0.5) (layer F.Cu) (net 2))
+  (segment (start 106.25 109.3575) (end 106.2625 109.37) (width 0.5) (layer F.Cu) (net 2))
+  (segment (start 106.25 107.39) (end 106.25 109.3575) (width 0.5) (layer F.Cu) (net 2))
+  (segment (start 106.43 113.76) (end 106.43 113.95) (width 0.25) (layer F.Cu) (net 3))
+  (segment (start 103.22 110.55) (end 106.43 113.76) (width 0.25) (layer F.Cu) (net 3))
+  (segment (start 112.82 110.489238) (end 112.82 109.57) (width 0.25) (layer F.Cu) (net 4))
+  (segment (start 112.82 111.19137) (end 112.82 110.489238) (width 0.25) (layer F.Cu) (net 4))
+  (segment (start 110.06137 113.95) (end 112.82 111.19137) (width 0.25) (layer F.Cu) (net 4))
+  (segment (start 108.93 113.95) (end 110.06137 113.95) (width 0.25) (layer F.Cu) (net 4))
+  (segment (start 117.98 110.4375) (end 116.41 110.4375) (width 0.25) (layer F.Cu) (net 4))
+  (segment (start 115.948388 109.975888) (end 115.385888 109.975888) (width 0.25) (layer F.Cu) (net 4))
+  (segment (start 116.41 110.4375) (end 115.948388 109.975888) (width 0.25) (layer F.Cu) (net 4))
+  (segment (start 114.98 109.57) (end 112.82 109.57) (width 0.25) (layer F.Cu) (net 4))
+  (segment (start 115.385888 109.975888) (end 114.98 109.57) (width 0.25) (layer F.Cu) (net 4))
+  (segment (start 116.41 108.8625) (end 117.98 108.8625) (width 0.25) (layer F.Cu) (net 5))
+  (segment (start 115.8475 108.3) (end 114.09 108.3) (width 0.25) (layer F.Cu) (net 5))
+  (segment (start 116.41 108.8625) (end 115.8475 108.3) (width 0.25) (layer F.Cu) (net 5))
+  (segment (start 109.74571 106.69429) (end 109.05 107.39) (width 0.25) (layer F.Cu) (net 5))
+  (segment (start 113.38429 106.69429) (end 109.74571 106.69429) (width 0.25) (layer F.Cu) (net 5))
+  (segment (start 114.09 107.4) (end 113.38429 106.69429) (width 0.25) (layer F.Cu) (net 5))
+  (segment (start 114.09 108.3) (end 114.09 107.4) (width 0.25) (layer F.Cu) (net 5))
+  (segment (start 119.2475 110.13) (end 117.98 108.8625) (width 0.25) (layer F.Cu) (net 5))
+  (segment (start 120.88 110.13) (end 119.2475 110.13) (width 0.25) (layer F.Cu) (net 5))
+  (segment (start 110.48 109.37) (end 111.55 108.3) (width 0.25) (layer F.Cu) (net 6))
+  (segment (start 107.8375 109.37) (end 110.48 109.37) (width 0.25) (layer F.Cu) (net 6))
+  (zone (net 1) (net_name "Net-(BT1-Pad1)") (layer F.Cu) (hatch edge 0.508)
+    (connect_pads (clearance 0.508))
+    (min_thickness 0.254)
+    (fill yes (arc_segments 32) (thermal_gap 0.508) (thermal_bridge_width 0.508))
+    (polygon
+      (pts
+        (xy 101.5 101.95) (xy 120.81 101.95) (xy 120.86 102.01) (xy 120.93 102.12) (xy 121.01 102.23)
+        (xy 121.09 102.36) (xy 121.19 102.48) (xy 121.27 102.62) (xy 121.39 102.78) (xy 121.49 102.96)
+        (xy 121.58 103.13) (xy 121.68 103.28) (xy 121.72 103.35) (xy 121.76 103.42) (xy 121.82 103.55)
+        (xy 121.91 103.71) (xy 122.07 104.04) (xy 122.18 104.27) (xy 122.37 104.72) (xy 122.47 105.02)
+        (xy 122.62 105.39) (xy 122.67 105.57) (xy 122.72 105.74) (xy 122.77 105.91) (xy 122.85 106.18)
+        (xy 122.89 106.35) (xy 122.95 106.64) (xy 123.02 106.96) (xy 123.08 107.24) (xy 123.1 107.44)
+        (xy 123.14 107.73) (xy 123.21 108.49) (xy 123.24 109.34) (xy 123.17 110.41) (xy 123.03 111.44)
+        (xy 122.77 112.5) (xy 122.23 114.03) (xy 121.95 114.63) (xy 121.6 115.28) (xy 121.1 116.06)
+        (xy 120.54 116.82) (xy 120.09 117.33) (xy 119.73 117.72) (xy 119.61 117.83) (xy 102.68 117.84)
+        (xy 102.24 117.36) (xy 101.45 116.42) (xy 101.22 116.08) (xy 101.03 115.79) (xy 100.82 115.47)
+        (xy 100.45 114.82) (xy 100.25 114.41) (xy 99.9 113.6) (xy 99.71 113.11) (xy 99.56 112.62)
+        (xy 99.45 112.2) (xy 99.29 111.49) (xy 99.21 111.03) (xy 99.11 110.11) (xy 99.07 109.57)
+        (xy 99.06 108.82) (xy 99.13 108) (xy 99.21 107.34) (xy 99.31 106.78) (xy 99.44 106.21)
+        (xy 99.63 105.56) (xy 99.91 104.79) (xy 100.13 104.26) (xy 100.42 103.7) (xy 100.84 102.91)
+        (xy 101.2 102.36)
+      )
+    )
+  )
+  (zone (net 1) (net_name "Net-(BT1-Pad1)") (layer B.Cu) (hatch edge 0.508)
+    (connect_pads (clearance 0.508))
+    (min_thickness 0.254)
+    (fill yes (arc_segments 32) (thermal_gap 0.508) (thermal_bridge_width 0.508))
+    (polygon
+      (pts
+        (xy 101.58 101.92) (xy 120.89 101.92) (xy 120.94 101.98) (xy 121.01 102.09) (xy 121.09 102.2)
+        (xy 121.17 102.33) (xy 121.27 102.45) (xy 121.35 102.59) (xy 121.47 102.75) (xy 121.57 102.93)
+        (xy 121.66 103.1) (xy 121.76 103.25) (xy 121.8 103.32) (xy 121.84 103.39) (xy 121.9 103.52)
+        (xy 121.99 103.68) (xy 122.15 104.01) (xy 122.26 104.24) (xy 122.45 104.69) (xy 122.55 104.99)
+        (xy 122.7 105.36) (xy 122.75 105.54) (xy 122.8 105.71) (xy 122.85 105.88) (xy 122.93 106.15)
+        (xy 122.97 106.32) (xy 123.03 106.61) (xy 123.1 106.93) (xy 123.16 107.21) (xy 123.18 107.41)
+        (xy 123.22 107.7) (xy 123.29 108.46) (xy 123.32 109.31) (xy 123.25 110.38) (xy 123.11 111.41)
+        (xy 122.85 112.47) (xy 122.31 114) (xy 122.03 114.6) (xy 121.68 115.25) (xy 121.18 116.03)
+        (xy 120.62 116.79) (xy 120.17 117.3) (xy 119.81 117.69) (xy 119.69 117.8) (xy 102.76 117.81)
+        (xy 102.32 117.33) (xy 101.53 116.39) (xy 101.3 116.05) (xy 101.11 115.76) (xy 100.9 115.44)
+        (xy 100.53 114.79) (xy 100.33 114.38) (xy 99.98 113.57) (xy 99.79 113.08) (xy 99.64 112.59)
+        (xy 99.53 112.17) (xy 99.37 111.46) (xy 99.29 111) (xy 99.19 110.08) (xy 99.15 109.54)
+        (xy 99.14 108.79) (xy 99.21 107.97) (xy 99.29 107.31) (xy 99.39 106.75) (xy 99.52 106.18)
+        (xy 99.71 105.53) (xy 99.99 104.76) (xy 100.21 104.23) (xy 100.5 103.67) (xy 100.92 102.88)
+        (xy 101.28 102.33)
+      )
+    )
+  )
+  (zone (net 0) (net_name "") (layer F.Cu) (hatch edge 0.508)
+    (connect_pads (clearance 0.508))
+    (min_thickness 0.254)
+    (fill yes (arc_segments 32) (thermal_gap 0.508) (thermal_bridge_width 0.508))
+    (polygon
+      (pts
+        (xy 105.28 107.81) (xy 104.16 109.21) (xy 104.26 110.89) (xy 106.31 112.62) (xy 108.3 112.8)
+        (xy 110.8 112.67) (xy 112.43 111.01) (xy 111.58 109.7) (xy 109.07 109.99) (xy 108.59 110.3)
+        (xy 105.57 110.3) (xy 105.27 110.2) (xy 105.3 108.51)
+      )
+    )
+  )
 )
